Commit message: copied urdf from simulation

File: src/lns_description/urdf/lns_robot.xacro (robot description, xacro)
@@ -4,5 +4,6 @@
      For more information, please see http://wiki.ros.org/sw_urdf_exporter -->
 <robot
-  name="lns_robot">
+  name="lns_robot" xmlns:xacro="http://ros.org/wiki/xacro">
+  <xacro:include filename="$(find lns_description)/urdf/lns_robot_control_transmission.xacro"/>
   <link name="base_footprint"/>
   <joint name="base_joint" type="fixed">
@@ -196,5 +197,5 @@
       link="steering_fl_link" />
     <axis
-      xyz="0 0 -1" />
+      xyz="0 0 1" />
     <limit
       lower="-2.1"
@@ -255,6 +256,5 @@
       xyz="-0.0003039 1 0" />
     <limit
-      lower="0"
-      effort="1.5"
+      effort="1000"
       velocity="20" />
   </joint>
@@ -309,5 +309,5 @@
       link="steering_fr_link" />
     <axis
-      xyz="0 0 -1" />
+      xyz="0 0 1" />
     <limit
       lower="-2.1"
@@ -366,8 +366,7 @@
       link="wheel_fr_link" />
     <axis
-      xyz="0.0023488 -1 0" />
-    <limit
-      lower="0"
-      effort="1.5"
+      xyz="0.0023488 1 0" />
+    <limit
+      effort="1000"
       velocity="20" />
   </joint>
@@ -422,5 +421,5 @@
       link="steering_br_link" />
     <axis
-      xyz="0 0 -1" />
+      xyz="0 0 1" />
     <limit
       lower="-2.1"
@@ -479,8 +478,7 @@
       link="wheel_br_link" />
     <axis
-      xyz="0.0023488 -1 0" />
-    <limit
-      lower="0"
-      effort="1.5"
+      xyz="0.0023488 1 0" />
+    <limit
+      effort="1000"
       velocity="20" />
   </joint>
@@ -535,5 +533,5 @@
       link="steering_bl_link" />
     <axis
-      xyz="0 0 -1" />
+      xyz="0 0 1" />
     <limit
       lower="-2.1"
@@ -594,6 +592,5 @@
       xyz="-0.0023488 1 0" />
     <limit
-      lower="0"
-      effort="1.5"
+      effort="1000"
       velocity="20" />
   </joint>
