Commit message: Fixed inertias

File: src/lns_description/urdf/lns_robot_sim.xacro (robot description, xacro)
@@ -20,12 +20,12 @@
         rpy="0 0 0" />
       <mass
-        value="115.323093862857" />
-      <inertia
-        ixx="30.5546981156896"
-        ixy="-0.00812450775540023"
-        ixz="0.0774264063877825"
-        iyy="38.3082783112508"
-        iyz="-0.141489346339812"
-        izz="51.8584316288848" />
+        value="400" />
+      <inertia
+        ixx="4.9554501882"
+        ixy="-0.0056002555"
+        ixz="-0.0304732818"
+        iyy="12.704705573"
+        iyz="-0.0509805808"
+        izz="10.448161117" />
     </inertial>
     <visual>
@@ -56,15 +56,15 @@
     <inertial>
       <origin
-        xyz="-0.720409053233766 0.00385628468290244 -0.975393530789188"
-        rpy="0 0 0" />
-      <mass
-        value="115.323093862857" />
-      <inertia
-        ixx="30.5546981156896"
-        ixy="-0.00812450775540023"
-        ixz="0.0774264063877825"
-        iyy="38.3082783112508"
-        iyz="-0.141489346339812"
-        izz="51.8584316288848" />
+        xyz="-0.00039033687859702 -1.53079096248954E-05 -0.000592327383379221"
+        rpy="0 0 0" />
+      <mass
+        value="0.195506924984229" />
+      <inertia
+        ixx="0.000195294443337896"
+        ixy="-5.19265291636756E-07"
+        ixz="-9.13195474661165E-09"
+        iyy="8.18066717719668E-05"
+        iyz="-5.5911022943428E-09"
+        izz="0.000248825415558086" />
     </inertial>
     <visual>
@@ -100,15 +100,15 @@
     <inertial>
       <origin
-        xyz="0.249441946765716 0.469559838074302 -0.480293530777087"
-        rpy="0 0 0" />
-      <mass
-        value="115.323093862857" />
-      <inertia
-        ixx="30.5546981156899"
-        ixy="-0.00812450775584025"
-        ixz="0.077426406419204"
-        iyy="38.3082783112512"
-        iyz="-0.141489346361371"
-        izz="51.8584316288841" />
+        xyz="0.00314804410618519 0.000886573216435982 -0.000493504453682236"
+        rpy="0 0 0" />
+      <mass
+        value="0.019931290489835" />
+      <inertia
+        ixx="6.18644586656033E-06"
+        ixy="5.13081146570535E-08"
+        ixz="-5.03594367346625E-08"
+        iyy="4.79889383234348E-06"
+        iyz="-5.65169719050544E-09"
+        izz="8.20604958309782E-06" />
     </inertial>
     <visual>
@@ -152,15 +152,15 @@
     <inertial>
       <origin
-        xyz="-0.500908053234454 -0.496143715201307 -0.252993530926179"
-        rpy="0 0 0" />
-      <mass
-        value="115.323093862857" />
-      <inertia
-        ixx="30.5546981156896"
-        ixy="-0.00812450775540023"
-        ixz="0.0774264063877825"
-        iyy="38.3082783112508"
-        iyz="-0.141489346339812"
-        izz="51.8584316288848" />
+        xyz="0.00018 -0.14605 -0.32841"
+        rpy="0 0 0" />
+      <mass
+        value="40" />
+      <inertia
+        ixx="0.0365913444"
+        ixy="-0.0013098542"
+        ixz="0.018645465"
+        iyy="0.1022477091"
+        iyz="-0.0003869004"
+        izz="0.0986761019" />
     </inertial>
     <visual>
@@ -209,15 +209,15 @@
     <inertial>
       <origin
-        xyz="-0.500915043003825 -0.473143716438484 0.180006469083252"
-        rpy="0 0 0" />
-      <mass
-        value="115.323093862857" />
-      <inertia
-        ixx="30.5546981156896"
-        ixy="-0.00812450775540023"
-        ixz="0.0774264063877825"
-        iyy="38.3082783112508"
-        iyz="-0.141489346339812"
-        izz="51.8584316288848" />
+        xyz="0.00001 0.02244 0.0"
+        rpy="1.57 0 0" />
+      <mass
+        value="8" />
+      <inertia
+        ixx="0.1109045059"
+        ixy="0.0000105925"
+        ixz="-0.0008373989"
+        iyy="0.1109470771"
+        iyz="0.0009631546"
+        izz="0.1871877734" />
     </inertial>
     <visual>
@@ -264,15 +264,15 @@
     <inertial>
       <origin
-        xyz="-0.50090805326955 0.501356284795344 -0.25299353052279"
-        rpy="0 0 0" />
-      <mass
-        value="115.323093862857" />
-      <inertia
-        ixx="30.5546981156896"
-        ixy="-0.00812450775540023"
-        ixz="0.0774264063877825"
-        iyy="38.3082783112508"
-        iyz="-0.141489346339812"
-        izz="51.8584316288848" />
+        xyz="-0.00048 0.14605 -0.32841"
+        rpy="0 0 0" />
+      <mass
+        value="40" />
+      <inertia
+        ixx="0.0365862618"
+        ixy="-0.0011755797"
+        ixz="-0.0186462173"
+        iyy="0.1022527916"
+        iyz="0.0003487706"
+        izz="0.0986761019" />
     </inertial>
     <visual>
@@ -321,15 +321,15 @@
     <inertial>
       <origin
-        xyz="-0.500854029674087 0.478356348066843 0.180006469468029"
-        rpy="0 0 0" />
-      <mass
-        value="115.323093862857" />
-      <inertia
-        ixx="30.5546981156896"
-        ixy="-0.00812450775540023"
-        ixz="0.0774264063877825"
-        iyy="38.3082783112508"
-        iyz="-0.141489346339812"
-        izz="51.8584316288848" />
+        xyz="0.00003 -0.02244 0.0"
+        rpy="1.57 0 0" />
+      <mass
+        value="8" />
+      <inertia
+        ixx="0.1108953254"
+        ixy="0.00000046192"
+        ixz="0.0000285233"
+        iyy="0.1109470816"
+        iyz="-0.0009634027"
+        izz="0.1871969494" />
     </inertial>
     <visual>
@@ -376,15 +376,15 @@
     <inertial>
       <origin
-        xyz="0.499091946762458 0.501356284680084 -0.252993530769525"
-        rpy="0 0 0" />
-      <mass
-        value="115.323093862857" />
-      <inertia
-        ixx="30.5546981156896"
-        ixy="-0.00812450775540023"
-        ixz="0.0774264063877825"
-        iyy="38.3082783112508"
-        iyz="-0.141489346339812"
-        izz="51.8584316288848" />
+        xyz="-0.00048 0.14605 -0.32841"
+        rpy="0 0 0" />
+      <mass
+        value="40" />
+      <inertia
+        ixx="0.0365862618"
+        ixy="-0.0011755797"
+        ixz="-0.0186462173"
+        iyy="0.1022527916"
+        iyz="0.0003487706"
+        izz="0.0986761019" />
     </inertial>
     <visual>
@@ -433,15 +433,15 @@
     <inertial>
       <origin
-        xyz="0.49914597035792 0.478356348127517 0.18000646923064"
-        rpy="0 0 0" />
-      <mass
-        value="115.323093862857" />
-      <inertia
-        ixx="30.5546981156896"
-        ixy="-0.00812450775540023"
-        ixz="0.0774264063877825"
-        iyy="38.3082783112508"
-        iyz="-0.141489346339812"
-        izz="51.8584316288848" />
+        xyz="0.00003 -0.02244 0"
+        rpy="1.57 0 0" />
+      <mass
+        value="8" />
+      <inertia
+        ixx="0.1108953254"
+        ixy="0.00000046192"
+        ixz="0.0000285233"
+        iyy="0.1109470816"
+        iyz="-0.0009634027"
+        izz="0.1871969494" />
     </inertial>
     <visual>
@@ -488,15 +488,15 @@
     <inertial>
       <origin
-        xyz="0.499091946761391 -0.49614371520285 -0.252993531055122"
-        rpy="0 0 0" />
-      <mass
-        value="115.323093862857" />
-      <inertia
-        ixx="30.5546981156896"
-        ixy="-0.00812450775540023"
-        ixz="0.0774264063877825"
-        iyy="38.3082783112508"
-        iyz="-0.141489346339812"
-        izz="51.8584316288848" />
+        xyz="0.00048 -0.14605 -0.32841"
+        rpy="0 0 0" />
+      <mass
+        value="40" />
+      <inertia
+        ixx="0.0365862618"
+        ixy="-0.0011755797"
+        ixz="0.0186462173"
+        iyy="0.1022527916"
+        iyz="-0.0003487706"
+        izz="0.0986761019" />
     </inertial>
     <visual>
@@ -545,15 +545,15 @@
     <inertial>
       <origin
-        xyz="0.499037923277592 -0.473143778824593 0.180006468954316"
-        rpy="0 0 0" />
-      <mass
-        value="115.323093862857" />
-      <inertia
-        ixx="30.5546981156896"
-        ixy="-0.00812450775540023"
-        ixz="0.0774264063877825"
-        iyy="38.3082783112508"
-        iyz="-0.141489346339812"
-        izz="51.8584316288848" />
+        xyz="-0.00003 0.02244 0.0"
+        rpy="1.57 0 0" />
+      <mass
+        value="8" />
+      <inertia
+        ixx="0.110904554"
+        ixy="0.0000106821"
+        ixz="-0.0008395766"
+        iyy="0.1109470336"
+        iyz="0.0009614396"
+        izz="0.1871877688" />
     </inertial>
     <visual>

Commit message: changed inertias to agilex robot

File: src/lns_description/urdf/lns_robot_sim.xacro (robot description, xacro)
@@ -17,15 +17,15 @@
     <inertial>
       <origin
-        xyz="-0.000908053234166831 0.00377583954880167 -0.11419353078418"
-        rpy="0 0 0" />
-      <mass
-        value="400" />
-      <inertia
-        ixx="4.9554501882"
-        ixy="-0.0056002555"
-        ixz="-0.0304732818"
-        iyy="12.704705573"
-        iyz="-0.0509805808"
-        izz="10.448161117" />
+        xyz="0 0 0"
+        rpy="0 0 0" />
+      <mass
+        value="17.59" />
+      <inertia
+        ixx="0.4691"
+        ixy="0"
+        ixz="0"
+        iyy="3.1076"
+        iyz="0"
+        izz="3.1076" />
     </inertial>
     <visual>
@@ -152,15 +152,15 @@
     <inertial>
       <origin
-        xyz="0.00018 -0.14605 -0.32841"
-        rpy="0 0 0" />
-      <mass
-        value="40" />
-      <inertia
-        ixx="0.0365913444"
-        ixy="-0.0013098542"
-        ixz="0.018645465"
-        iyy="0.1022477091"
-        iyz="-0.0003869004"
-        izz="0.0986761019" />
+        xyz="0 0 0"
+        rpy="0 0 0" />
+      <mass
+        value="0.29" />
+      <inertia
+        ixx="5.3495E-4"
+        ixy="0"
+        ixz="0"
+        iyy="5.3495E-4"
+        iyz="0"
+        izz="4.3069E-4" />
     </inertial>
     <visual>
@@ -209,15 +209,15 @@
     <inertial>
       <origin
-        xyz="0.00001 0.02244 0.0"
+        xyz="0 0.023 0"
         rpy="1.57 0 0" />
       <mass
-        value="8" />
-      <inertia
-        ixx="0.1109045059"
-        ixy="0.0000105925"
-        ixz="-0.0008373989"
-        iyy="0.1109470771"
-        iyz="0.0009631546"
-        izz="0.1871877734" />
+        value="1.1" />
+      <inertia
+        ixx="0.0133"
+        ixy="0"
+        ixz="0"
+        iyy="0.0133"
+        iyz="0"
+        izz="0.022" />
     </inertial>
     <visual>
@@ -264,15 +264,15 @@
     <inertial>
       <origin
-        xyz="-0.00048 0.14605 -0.32841"
-        rpy="0 0 0" />
-      <mass
-        value="40" />
-      <inertia
-        ixx="0.0365862618"
-        ixy="-0.0011755797"
-        ixz="-0.0186462173"
-        iyy="0.1022527916"
-        iyz="0.0003487706"
-        izz="0.0986761019" />
+        xyz="0 0 0"
+        rpy="0 0 0" />
+      <mass
+        value="0.29" />
+      <inertia
+        ixx="5.3495E-4"
+        ixy="0"
+        ixz="0"
+        iyy="5.3495E-4"
+        iyz="0"
+        izz="4.3069E-4" />
     </inertial>
     <visual>
@@ -321,15 +321,15 @@
     <inertial>
       <origin
-        xyz="0.00003 -0.02244 0.0"
+        xyz="0 -0.023 0"
         rpy="1.57 0 0" />
       <mass
-        value="8" />
-      <inertia
-        ixx="0.1108953254"
-        ixy="0.00000046192"
-        ixz="0.0000285233"
-        iyy="0.1109470816"
-        iyz="-0.0009634027"
-        izz="0.1871969494" />
+        value="1.1" />
+      <inertia
+        ixx="0.0133"
+        ixy="0"
+        ixz="0"
+        iyy="0.0133"
+        iyz="0"
+        izz="0.022" />
     </inertial>
     <visual>
@@ -376,15 +376,15 @@
     <inertial>
       <origin
-        xyz="-0.00048 0.14605 -0.32841"
-        rpy="0 0 0" />
-      <mass
-        value="40" />
-      <inertia
-        ixx="0.0365862618"
-        ixy="-0.0011755797"
-        ixz="-0.0186462173"
-        iyy="0.1022527916"
-        iyz="0.0003487706"
-        izz="0.0986761019" />
+        xyz="0 0 0"
+        rpy="0 0 0" />
+      <mass
+        value="0.29" />
+      <inertia
+        ixx="5.3495E-4"
+        ixy="0"
+        ixz="0"
+        iyy="5.3495E-4"
+        iyz="0"
+        izz="4.3069E-4" />
     </inertial>
     <visual>
@@ -433,15 +433,15 @@
     <inertial>
       <origin
-        xyz="0.00003 -0.02244 0"
+        xyz="0 -0.023 0"
         rpy="1.57 0 0" />
       <mass
-        value="8" />
-      <inertia
-        ixx="0.1108953254"
-        ixy="0.00000046192"
-        ixz="0.0000285233"
-        iyy="0.1109470816"
-        iyz="-0.0009634027"
-        izz="0.1871969494" />
+        value="1.1" />
+      <inertia
+        ixx="0.0133"
+        ixy="0"
+        ixz="0"
+        iyy="0.0133"
+        iyz="0"
+        izz="0.022" />
     </inertial>
     <visual>
@@ -488,15 +488,15 @@
     <inertial>
       <origin
-        xyz="0.00048 -0.14605 -0.32841"
-        rpy="0 0 0" />
-      <mass
-        value="40" />
-      <inertia
-        ixx="0.0365862618"
-        ixy="-0.0011755797"
-        ixz="0.0186462173"
-        iyy="0.1022527916"
-        iyz="-0.0003487706"
-        izz="0.0986761019" />
+        xyz="0 0 0"
+        rpy="0 0 0" />
+      <mass
+        value="0.29" />
+      <inertia
+        ixx="5.3495E-4"
+        ixy="0"
+        ixz="0"
+        iyy="5.3495E-4"
+        iyz="0"
+        izz="4.3069E-4" />
     </inertial>
     <visual>
@@ -545,15 +545,15 @@
     <inertial>
       <origin
-        xyz="-0.00003 0.02244 0.0"
+        xyz="0 0.023 0"
         rpy="1.57 0 0" />
       <mass
-        value="8" />
-      <inertia
-        ixx="0.110904554"
-        ixy="0.0000106821"
-        ixz="-0.0008395766"
-        iyy="0.1109470336"
-        iyz="0.0009614396"
-        izz="0.1871877688" />
+        value="1.1" />
+      <inertia
+        ixx="0.0133"
+        ixy="0"
+        ixz="0"
+        iyy="0.0133"
+        iyz="0"
+        izz="0.022" />
     </inertial>
     <visual>
